File: PCB/main-board/main-board.kicad_sch (KiCad schematic)
At the start: 91 parts, among them J1 AudioJack2_Ground_Switch, J2 AudioJack2_Ground_Switch, J3 AudioJack2_Ground_Switch, J4 AudioJack2_Ground_Switch, J5 AudioJack2_Ground_Switch, J6 Conn_01x14, J7 Conn_01x03, Q1 Si1308EDL, Q10 Si1308EDL, Q11 DMG2305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

Commit message: Non-populate 3-pin header.
Parts:
- J7: now not fitted; now left out of the parts list
Changed lines of the file:
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@@
 		(unit 1)
 		(exclude_from_sim no)
-		(in_bom yes)
+		(in_bom no)
 		(on_board yes)
-		(dnp no)
+		(dnp yes)
 		(property "Reference" "J7"
 			(at 83.82 39.37 0)
